File: adapter_board/YYSJ_2.1''_knob/YYSJ_2.1''_knob.kicad_sch (KiCad schematic)
At the start: 12 parts, among them J1 USB_C_Receptacle_USB2.0, J2 FPC 10, J3 Conn_01x10

Commit message: adapter_board.YYSJ_2.1''knob: finish electric
Parts:
- J3: footprint Connector_PinHeader_2.54mm:PinHeader_1x10_P2.54mm_Vertical -> Connector_PinHeader_2.54mm:PinHeader_1x10_P2.54mm_Horizontal
Changed lines of the file:
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@@
       (effects (font (size 1.27 1.27)) (justify left))
     )
-    (property "Footprint" "Connector_PinHeader_2.54mm:PinHeader_1x10_P2.54mm_Vertical" (id 2) (at 177.8 80.01 0)
+    (property "Footprint" "Connector_PinHeader_2.54mm:PinHeader_1x10_P2.54mm_Horizontal" (id 2) (at 177.8 80.01 0)
       (effects (font (size 1.27 1.27)) hide)
     )
@@
     )
     (path "/f1e19be3-64f5-4d01-96f7-ba7767e1c4a1"
-      (reference "J3") (unit 1) (value "Conn_01x10") (footprint "Connector_PinHeader_2.54mm:PinHeader_1x10_P2.54mm_Vertical")
+      (reference "J3") (unit 1) (value "Conn_01x10") (footprint "Connector_PinHeader_2.54mm:PinHeader_1x10_P2.54mm_Horizontal")
     )
     (path "/1c70287e-8da0-4aeb-b002-ee811cbf6064"
