File: adapter_board/YYSJ_2.1''_knob/YYSJ_2.1''_knob.kicad_pcb (KiCad board)
At the start: 2 copper layers, 12 parts, among them J1 USB_C_Receptacle_USB2.0, J2 FPC 10, J3 Conn_01x10

Commit message: adapter_board.YYSJ_2.1''knob: finish electric
Parts:
- J2: moved to B.Cu
- J3: footprint Connector_PinHeader_2.54mm:PinHeader_1x10_P2.54mm_Vertical -> Connector_PinHeader_2.54mm:PinHeader_1x10_P2.54mm_Horizontal
- moved J3 275.3 mm to (60.6, 141.0), turned to 180 degrees
- moved J2 224.6 mm to (71.0, 129.5), turned to -90 degrees
- moved D5 147.0 mm to (68.3, 93.5)
- moved R3 145.7 mm to (64.8, 93.5)
- moved C1 137.2 mm to (71.4, 95.0), turned to 90 degrees
- moved D4 136.6 mm to (66.8, 96.5), turned to 180 degrees
- moved D3 115.6 mm to (61.9, 96.0), turned to -90 degrees
- moved R2 115.4 mm to (58.0, 107.4)
- moved D2 112.8 mm to (61.9, 102.4), turned to 90 degrees
- moved R1 109.8 mm to (58.0, 94.2)
- moved D1 107.5 mm to (61.9, 99.8), turned to -90 degrees
- moved J1 81.8 mm to (54.2, 100.8), turned to -90 degrees
Routing:
- net /VCC5V: track 0.00 -> 62.3 mm, vias 0 -> 1
- net /USB_D-: track 0.00 -> 60.4 mm, vias 0 -> 3
- net /USB_D+: track 0.00 -> 60.4 mm, vias 0 -> 1
- net Net-(D3-Pad2): track 0.00 -> 13.0 mm
- net Net-(J2-Pad9): track 0.00 -> 11.5 mm
- net Net-(J2-Pad3): track 0.00 -> 10.6 mm
- net Net-(J2-Pad4): track 0.00 -> 9.77 mm
- net Net-(J2-Pad7): track 0.00 -> 9.77 mm
- net Net-(J2-Pad5): track 0.00 -> 8.93 mm
- net Net-(J2-Pad6): track 0.00 -> 8.92 mm
- net Net-(J1-PadB5): track 0.00 -> 8.34 mm, vias 0 -> 2
- net Net-(J1-PadA5): track 0.00 -> 8.15 mm, vias 0 -> 2
- net Net-(D5-Pad1): track 0.00 -> 1.94 mm
- added copper zone on B.Cu, net /VCC5V
- added copper zone on F.Cu, net /VCC5V
- added copper zone on F.Cu, net Net-(D3-Pad2)
Other:
- board outline added: 80 x 80 mm
- board text added: "5V"
- board text added: "ADC"
- board text added: "GND"
- board text added: "RST"
- board text added: "RXD"
- board text added: "TXD"
- board text added: "USB+"
- board text added: "USB-"

Commit message: adapter_board.YYSJ_2.1''knob: finish
Parts:
- added G***: ESP_LOGO, LOGO:LOGO, F.Cu at (84.9, 161.6)
- added REF**: KiCad-Logo2_5mm_SilkScreen, Symbol:KiCad-Logo2_5mm_SilkScreen, F.Cu at (109.3, 161.1)
- moved D1 4.58 mm to (61.8, 104.4)
- moved D3 4.58 mm to (61.8, 100.6)
- moved C1 4.58 mm to (71.3, 99.6)
- moved D2 4.58 mm to (61.8, 106.9)
- moved D4 4.58 mm to (66.6, 101.1)
- moved D5 4.58 mm to (68.2, 98.0)
- moved R1 4.58 mm to (57.9, 98.8)
- moved R2 4.58 mm to (57.9, 112.0)
- moved R3 4.58 mm to (64.6, 98.0)
- moved J1 4.58 mm to (54.1, 105.4)
Routing:
- net /VCC5V: track 62.3 -> 57.7 mm
- net /USB_D-: track 60.4 -> 58.6 mm
- net /USB_D+: track 60.4 -> 58.6 mm
- added copper zone on B.Cu, net GND
- added copper zone on F.Cu, net GND
Other:
- board size 80 x 80 mm -> 81 x 81 mm
